File: 02_pcb_interface_board_design/kicad_project_files/elevator_io_interface_board.kicad_pcb (KiCad board)
At the start: 2 copper layers, 47 parts, among them J1 Power Input, J10 MCU Output Header, J11 Motor UP Output, J12 Motor DOWN Output, J13 Door OPEN Output, J14 Door CLOSE Output, J2 MCU Input Header, J3 Floor 1 Button, J4 Floor 2 Button, J5 Floor 3 Button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

Commit message: PCB Finalize!
Parts:
- removed C1: 100nF, Capacitor_THT:C_Disc_D5.0mm_W2.5mm_P5.00mm
- added C3: 10uF, Capacitor_THT:CP_Radial_D5.0mm_P2.50mm, F.Cu at (77.5, 86.6)
- added C4: 10uF, Capacitor_THT:CP_Radial_D5.0mm_P2.50mm, F.Cu at (77.6, 93.3)
- added C5: 10uF, Capacitor_THT:CP_Radial_D5.0mm_P2.50mm, F.Cu at (90.7, 103.8)
- added C6: 100nF, Capacitor_THT:C_Disc_D5.0mm_W2.5mm_P5.00mm, F.Cu at (103.2, 116.4)
- added C7: 100nF, Capacitor_THT:C_Disc_D5.0mm_W2.5mm_P5.00mm, F.Cu at (103.3, 123.9)
- added C8: 100nF, Capacitor_THT:C_Disc_D5.0mm_W2.5mm_P5.00mm, F.Cu at (98.2, 108.7)
- added C9: 100nF, Capacitor_THT:C_Disc_D5.0mm_W2.5mm_P5.00mm, F.Cu at (103.1, 108.5)
- added J15: SWD_IO, Connector_PinHeader_2.54mm:PinHeader_1x04_P2.54mm_Vertical, F.Cu at (112.6, 111.7)
- added R16: 10k, Resistor_THT:R_Axial_DIN0207_L6.3mm_D2.5mm_P7.62mm_Horizontal, F.Cu at (76.9, 107.9)
- added R17: 10k, Resistor_THT:R_Axial_DIN0207_L6.3mm_D2.5mm_P7.62mm_Horizontal, F.Cu at (101.2, 89.2)
- added SW1: SW_Push, Button_Switch_THT:SW_PUSH_6mm, F.Cu at (77.8, 112.4)
- added SW2: SW_SPDT, Button_Switch_SMD:SW_SPDT_PCM12, F.Cu at (101.9, 78.9)
- added U1: STM32F103C8T6, Package_QFP:LQFP-48_7x7mm_P0.5mm, F.Cu at (93.0, 114.2)
- added U2: AMS1117-3.3, Package_TO_SOT_SMD:SOT-223-3_TabPin2, F.Cu at (90.4, 93.5)
- J6: value Door Obstruction Sensor -> Door Sensor
- J7: value Emergency Stop Input -> Emergency Stop
- moved K1 141.1 mm to (144.6, 164.6)
- moved Q1 121.8 mm to (126.6, 171.0), turned to 90 degrees
- moved K2 115.8 mm to (144.7, 144.3)
- moved LED1 115.0 mm to (127.3, 160.2), turned to 180 degrees
- moved R8 108.4 mm to (140.7, 164.4), turned to 180 degrees
- moved K3 98.6 mm to (144.7, 125.0)
- moved Q2 96.7 mm to (126.1, 150.7), turned to 90 degrees
- moved D1 94.4 mm to (141.1, 170.9), turned to 180 degrees
- moved J2 93.3 mm to (83.2, 145.3), turned to 90 degrees
- moved K4 92.8 mm to (144.3, 105.8)
- moved R12 92.2 mm to (140.7, 158.4), turned to 180 degrees
- moved LED2 89.9 mm to (127.3, 139.9), turned to 180 degrees
- moved R1 85.4 mm to (80.6, 137.0), turned to 90 degrees
- moved R9 85.3 mm to (132.7, 144.7)
- moved R2 82.0 mm to (85.2, 137.0), turned to 90 degrees
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Connections:
- J10 pad 5: +5V -> +3.3V
- J2 pad 1: +5V -> +3.3V
- J3 pad 1: +5V -> +3.3V
- J4 pad 1: +5V -> +3.3V
- J5 pad 1: +5V -> +3.3V
- J6 pad 1: +5V -> +3.3V
- J7 pad 1: +5V -> +3.3V
- J8 pad 1: +5V -> +3.3V
- J9 pad 1: +5V -> +3.3V
Other:
- board outline added: 94.2 x 102 mm

Commit message: PCB Design finalized!
Parts:
- moved K1 0.19 mm to (144.8, 164.5)
Changed lines of the file:
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@@
 	(footprint "Relay_THT:Relay_SPDT_SANYOU_SRD_Series_Form_C"
 		(layer "F.Cu")
-		(at 144.592 164.5506)
+		(at 144.7858 164.5364)
 		(descr "relay Sanyou SRD series Form C http://www.sanyourelay.ca/public/products/pdf/SRD.pdf")
 		(tags "relay Sanyu SRD form C")
