File: 02_pcb_interface_board_design/kicad_project_files/elevator_io_interface_board.kicad_sch (KiCad schematic)
At the start: 48 parts, among them J1 Power Input, J10 MCU Output Header, J11 Motor UP Output, J12 Motor DOWN Output, J13 Door OPEN Output, J14 Door CLOSE Output, J2 MCU Input Header, J3 Floor 1 Button, J4 Floor 2 Button, J5 Floor 3 Button, J6 Door Obstruction Sensor, J7 Emergency Stop Input, J8 Upper Limit Switch, J9 Lower Limit Switch, K1 Relay_SPDT, K2 Relay_SPDT, K3 Relay_SPDT, K4 Relay_SPDT, Q1 2N2222, Q2 2N2222, Q3 2N2222, Q4 2N2222, U1 STM32F103C8Tx

Commit message: PCB Finalize!
Parts:
- removed C1: 100nF, Capacitor_THT:C_Disc_D5.0mm_W2.5mm_P5.00mm, symbol Device:C
- added C3, C4, C5: 10uF, Capacitor_THT:CP_Radial_D5.0mm_P2.50mm, symbol Device:C
- added C6, C7, C8, C9: 100nF, Capacitor_THT:C_Disc_D5.0mm_W2.5mm_P5.00mm, symbol Device:C
- added J15: SWD_IO, Connector_PinHeader_2.54mm:PinHeader_1x04_P2.54mm_Vertical, symbol Connector:Conn_01x04_Pin
- added R16, R17: 10k, Resistor_THT:R_Axial_DIN0207_L6.3mm_D2.5mm_P7.62mm_Horizontal, symbol Device:R
- added SW1: SW_Push, Button_Switch_THT:SW_PUSH_6mm, symbol Switch:SW_Push
- added SW2: SW_SPDT, Button_Switch_SMD:SW_SPDT_PCM12, symbol Switch:SW_SPDT
- added U2: AMS1117-3.3, Package_TO_SOT_SMD:SOT-223-3_TabPin2, symbol Regulator_Linear:AMS1117-3.3
- U1: value STM32F103C8Tx -> STM32F103C8T6
Connections:
- net +5V: now also C3.1, U2.3 (VI); no longer J10.5 (Pin_5), J2.1 (Pin_1), J3.1 (Pin_1), J4.1 (Pin_1), J5.1 (Pin_1), J6.1 (Pin_1), J7.1 (Pin_1), J8.1 (Pin_1), J9.1 (Pin_1)
- net DOOR_CLOSE_CMD: now also U1.39 (PB3)
- net DOOR_OBSTRUCTION: now also U1.13 (PA3)
- net DOOR_OPEN_CMD: now also U1.20 (PB2)
- net EMERGENCY_STOP: now also U1.14 (PA4)
- net FLOOR_1_REQ: now also U1.10 (PA0)
- net FLOOR_2_REQ: now also U1.11 (PA1)
- net FLOOR_3_REQ: now also U1.12 (PA2)
- net GND: now also U1.23 (VSS), U1.35 (VSS), U1.47 (VSS), U1.8 (VSSA), C3.2, C4.2, C5.2, C6.1, C7.1, C8.1, C9.1, J15.4 (Pin_4), SW1.1, SW2.1 (A), U2.1 (GND)
- net LIMIT_DOWN: now also U1.16 (PA6)
- net LIMIT_UP: now also U1.15 (PA5)
- net MOTOR_DOWN_CMD: now also U1.19 (PB1)
- net MOTOR_UP_CMD: now also U1.18 (PB0)
- net +3.3V: now reaches U1.1 (VBAT)
- net +3.3V: now also J10.5 (Pin_5), J2.1 (Pin_1), J3.1 (Pin_1), J4.1 (Pin_1), J5.1 (Pin_1), J6.1 (Pin_1), J7.1 (Pin_1), J8.1 (Pin_1), J9.1 (Pin_1), U1.24 (VDD), U1.36 (VDD), U1.48 (VDD), C4.1, C5.1, C6.2, C7.2, C8.2, C9.2, J15.1 (Pin_1), R16.1, SW2.3 (C), U2.2 (VO)
- net SWDIO: now reaches U1.34 (PA13)
- net SWDIO: now also J15.2 (Pin_2)
- net SWCLK: now reaches U1.37 (PA14)
- net SWCLK: now also J15.3 (Pin_3)
- net at U1.44 (BOOT0): now also R17.2
- net at U1.7 (NRST): now also R16.2, SW1.2
- new net: R17.1, SW2.2 (B)
- no-connect marks 6 -> 30
Other:
- moved on the sheet: C2, D1, D2, D3, D4, J1, J10, J11, J12, J13, J14, J2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

Commit message: PCB updated!
Parts:
- removed K1: Relay_SPDT, Relay_THT:Relay_SPDT_SANYOU_SRD_Series_Form_C, symbol Relay:Relay_SPDT
- added K1: Relay-LYCA005x, Relay_THT:Relay_SPDT_Fujitsu_FTR-LYCA005x_FormC_Vertical, symbol Relay:Fujitsu_FTR-LYCA005x
- K2, K3, K4: value Relay_SPDT -> Relay-LYCA005x; footprint Relay_THT:Relay_SPDT_SANYOU_SRD_Series_Form_C -> Relay_THT:Relay_SPDT_Fujitsu_FTR-LYCA005x_FormC_Vertical
Connections:
- net +12V: now also K1.11, K1.A1
- net at D1.2 (A), Q1.2 (C): now also K1.A2
- net at J11.1 (Pin_1): now also K1.14
Changed lines of the file:
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@@
 	(paper "A4")
 	(junction
+		(at 76.2 76.2)
+		(diameter 0)
+		(color 0 0 0 0)
+	)
+	(junction
 		(at 102.87 113.03)
 		(diameter 0)
@@
 	)
 	(junction
-		(at 76.2 102.87)
-		(diameter 0)
-		(color 0 0 0 0)
-	)
-	(junction
 		(at 26.67 163.83)
 		(diameter 0)
@@
 	)
 	(junction
-		(at 76.2 76.2)
-		(diameter 0)
-		(color 0 0 0 0)
-	)
-	(junction
 		(at 214.63 124.46)
 		(diameter 0)
@@
 	)
 	(junction
+		(at 76.2 102.87)
+		(diameter 0)
+		(color 0 0 0 0)
+	)
+	(junction
 		(at 29.21 38.1)
 		(diameter 0)
@@
 	(wire
 		(pts
+			(xy 76.2 76.2) (xy 76.2 82.55)
+		)
+		(stroke
+			(width 0)
+			(type default)
+		)
+	)
+	(wire
+		(pts
 			(xy 15.24 38.1) (xy 15.24 30.48)
 		)
@@
 	(wire
 		(pts
-			(xy 76.2 76.2) (xy 76.2 82.55)
-		)
-		(stroke
-			(width 0)
-			(type default)
-		)
-	)
-	(wire
-		(pts
 			(xy 190.5 82.55) (xy 187.96 82.55)
 		)
@@
 	(wire
 		(pts
-			(xy 76.2 97.79) (xy 76.2 102.87)
-		)
-		(stroke
-			(width 0)
-			(type default)
-		)
-	)
-	(wire
-		(pts
 			(xy 130.81 49.53) (xy 130.81 50.8)
 		)
@@
 	(wire
 		(pts
-			(xy 86.36 97.79) (xy 86.36 102.87)
-		)
-		(stroke
-			(width 0)
-			(type default)
-		)
-	)
-	(wire
-		(pts
 			(xy 76.2 158.75) (xy 76.2 163.83)
 		)
@@
 	(wire
 		(pts
+			(xy 76.2 97.79) (xy 76.2 102.87)
+		)
+		(stroke
+			(width 0)
+			(type default)
+		)
+	)
+	(wire
+		(pts
 			(xy 29.21 119.38) (xy 26.67 119.38)
 		)
@@
 	(wire
 		(pts
+			(xy 86.36 97.79) (xy 86.36 102.87)
+		)
+		(stroke
+			(width 0)
+			(type default)
+		)
+	)
+	(wire
+		(pts
 			(xy 76.2 119.38) (xy 76.2 124.46)
 		)
@@
 	)
 	(symbol
+		(lib_id "Relay:Fujitsu_FTR-LYCA005x")
+		(at 81.28 90.17 0)
+		(unit 1)
+		(body_style 1)
+		(exclude_from_sim no)
+		(in_bom yes)
+		(on_board yes)
+		(in_pos_files yes)
+		(dnp no)
+		(fields_autoplaced yes)
+		(property "Reference" "K1"
+			(at 92.71 88.8999 0)
+			(show_name no)
+			(do_not_autoplace no)
+			(effects
+				(font
+					(size 1.27 1.27)
+				)
+				(justify left)
+			)
+		)
+		(property "Value" "Relay-LYCA005x"
+			(at 92.71 91.4399 0)
+			(show_name no)
+			(do_not_autoplace no)
+			(effects
+				(font
+					(size 1.27 1.27)
+				)
+				(justify left)
+			)
+		)
+		(property "Footprint" "Relay_THT:Relay_SPDT_Fujitsu_FTR-LYCA005x_FormC_Vertical"
+			(at 92.71 91.44 0)
+			(hide yes)
+			(show_name no)
+			(do_not_autoplace no)
+			(effects
+				(font
+					(size 1.27 1.27)
+				)
+				(justify left)
+			)
+		)
+		(property "Datasheet" "https://www.fujitsu.com/sg/imagesgig5/ftr-ly.pdf"
+			(at 97.79 93.98 0)
+			(hide yes)
+			(show_name no)
+			(do_not_autoplace no)
+			(effects
+				(font
+					(size 1.27 1.27)
+				)
+				(justify left)
+			)
+		)
+		(property "Description" "Relay, SPDT Form C, vertical mount, 5-60V coil, 6A, 250VAC, 28 x 5 x 15mm"
+			(at 81.28 90.17 0)
+			(hide yes)
+			(show_name no)
+			(do_not_autoplace no)
+			(effects
+				(font
+					(size 1.27 1.27)
+				)
+			)
+		)
+		(pin "14"
+		)
+		(pin "A2"
+		)
+		(pin "A1"
+		)
+		(pin "11"
+		)
+		(pin "12"
+		)
+		(instances
+			(project "elevator_io_interface_board"
+				(path "/2a0a01bd-921b-461d-b5b7-63f5d162ec94"
+					(reference "K1")
+					(unit 1)
+				)
+			)
+		)
+	)
+	(symbol
 		(lib_id "Device:R")
 		(at 43.18 113.03 90)
@@
 			)
 		)
-		(property "Value" "Relay_SPDT"
+		(property "Value" "Relay-LYCA005x"
 			(at 43.18 91.4399 0)
 			(show_name no)
@@
 			)
 		)
-		(property "Footprint" "Relay_THT:Relay_SPDT_SANYOU_SRD_Series_Form_C"
+		(property "Footprint" "Relay_THT:Relay_SPDT_Fujitsu_FTR-LYCA005x_FormC_Vertical"
 			(at 43.18 91.44 0)
 			(hide yes)
@@
 	)
 	(symbol
-		(lib_id "Relay:Relay_SPDT")
-		(at 81.28 90.17 0)
-		(unit 1)
-		(body_style 1)
-		(exclude_from_sim no)
-		(in_bom yes)
-		(on_board yes)
-		(in_pos_files yes)
-		(dnp no)
-		(fields_autoplaced yes)
-		(property "Reference" "K1"
-			(at 92.71 88.8999 0)
-			(show_name no)
-			(do_not_autoplace no)
-			(effects
-				(font
-					(size 1.27 1.27)
-				)
-				(justify left)
-			)
-		)
-		(property "Value" "Relay_SPDT"
-			(at 92.71 91.4399 0)
-			(show_name no)
-			(do_not_autoplace no)
-			(effects
-				(font
-					(size 1.27 1.27)
-				)
-				(justify left)
-			)
-		)
-		(property "Footprint" "Relay_THT:Relay_SPDT_SANYOU_SRD_Series_Form_C"
-			(at 92.71 91.44 0)
-			(hide yes)
-			(show_name no)
-			(do_not_autoplace no)
-			(effects
-				(font
-					(size 1.27 1.27)
-				)
-				(justify left)
-			)
-		)
-		(property "Datasheet" ""
-			(at 81.28 90.17 0)
-			(hide yes)
-			(show_name no)
-			(do_not_autoplace no)
-			(effects
-				(font
-					(size 1.27 1.27)
-				)
-			)
-		)
-		(property "Description" "Relay SPDT, monostable, EN50005"
-			(at 81.28 90.17 0)
-			(hide yes)
-			(show_name no)
-			(do_not_autoplace no)
-			(effects
-				(font
-					(size 1.27 1.27)
-				)
-			)
-		)
-		(pin "11"
-		)
-		(pin "14"
-		)
-		(pin "A1"
-		)
-		(pin "12"
-		)
-		(pin "A2"
-		)
-		(instances
-			(project "elevator_io_interface_board"
-				(path "/2a0a01bd-921b-461d-b5b7-63f5d162ec94"
-					(reference "K1")
-					(unit 1)
-				)
-			)
-		)
-	)
-	(symbol
 		(lib_id "MCU_ST_STM32F1:STM32F103C8Tx")
 		(at 170.18 105.41 0)
@@
 			)
 		)
-		(property "Value" "Relay_SPDT"
+		(property "Value" "Relay-LYCA005x"
 			(at 92.71 152.3999 0)
 			(show_name no)
@@
 			)
 		)
-		(property "Footprint" "Relay_THT:Relay_SPDT_SANYOU_SRD_Series_Form_C"
+		(property "Footprint" "Relay_THT:Relay_SPDT_Fujitsu_FTR-LYCA005x_FormC_Vertical"
 			(at 92.71 152.4 0)
 			(hide yes)
@@
 			)
 		)
-		(property "Value" "Relay_SPDT"
+		(property "Value" "Relay-LYCA005x"
 			(at 43.18 152.3999 0)
 			(show_name no)
@@
 			)
 		)
-		(property "Footprint" "Relay_THT:Relay_SPDT_SANYOU_SRD_Series_Form_C"
+		(property "Footprint" "Relay_THT:Relay_SPDT_Fujitsu_FTR-LYCA005x_FormC_Vertical"
 			(at 43.18 152.4 0)
 			(hide yes)
